File: mindaq_pcb/mindaq.kicad_pcb (KiCad board)
At the start: 2 copper layers, 41.8 x 29 mm, 55 parts, among them J1 Adafruit 4383 Color TFT + μSD, J2 6-axis F/T, J3 VMEAS+, J6 SHUNT, U1 ADS131M08IPBSR, U2 ESP32S3, U3 REF5025AIDR, U4 OPA2333AIDR, U5 SRV05-4, U6 SRV05-4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

Commit message: generate production files for jlcpcb
Parts:
- C17: value 2.2nF -> 1nF
- R2, R3, R4, R7: value 10k -> 47k
