File: mindaq_pcb/mindaq.kicad_sch (KiCad schematic)
At the start: 55 parts, among them J1 Adafruit 4383 Color TFT + μSD, J2 6-axis F/T, J3 VMEAS+, J6 SHUNT, U1 ADS131M08IPBSR, U2 ESP32S3, U3 REF5025AIDR, U4 OPA2333AIDR, U5 SRV05-4, U6 SRV05-4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

Commit message: generate production files for jlcpcb
Parts:
- C1, C11, C2, C3, C4, C7: LCSC (none) -> C52923
- C12, C13, C14, C15, C16, C18, C8: LCSC (none) -> C15195
- C17: value 2.2nF -> 1nF; LCSC (none) -> C1523
- C5: LCSC (none) -> C15525
- C6: LCSC (none) -> C16772
- C9: LCSC (none) -> C307331
- R1: LCSC (none) -> C25105
- R10, R11, R12, R13, R14, R15, R16, R17, R20, R21, R5, R6, R8, R9: LCSC (none) -> C25076
- R18: LCSC (none) -> C25792
- R19: LCSC (none) -> C4109
- R2, R3, R4, R7: value 10k -> 47k; LCSC (none) -> C25792
- U5, U6: now not fitted; now left out of the parts list
Other:
- note added: "bus voltage measurement ≤29.4V input range is ±1.2V scale 24.5x RC filt about 80kHz"
- note added: "current measurement RC antialias about 80kHz"
- note removed: "bus voltage measurement ≤29.4V input range is ±1.2V scale 24.5x RC filt about 30kHz"
- note removed: "current measurement"
